File: VECTAR-PSU-Rev1a.kicad_pcb (KiCad board)
At the start: 2 copper layers, 65 parts, among them J1 XT60PW-M, J2 XT60PW-M, J3 Conn_01x02_Socket, J5 Conn_01x06_Socket, J6 XT90PW-M, Q1 2N7002, Q2 IRFB7437, Q3 IRFB7437, SW2 RA1113112R, U1 LM74502DDFR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

Commit message: PCB Rev 1 Complete
Parts:
- added TP12: TestPoint, PSU-Rev1:KEYSTONE_5002, F.Cu at (119.0, 78.0)
- F1: footprint PSU-Rev1:0498150.M -> PSU-Rev1:3-140-178
- Q1, R3, R4, R5, R6: moved to B.Cu
- R1: value 2.27k -> 1.9k; moved to B.Cu
- moved TP2 158.9 mm to (185.0, 25.0)
- moved D4 158.0 mm to (189.3, 69.0), turned to 180 degrees
- moved TP8 155.5 mm to (184.8, 75.7)
- moved TP6 145.8 mm to (177.0, 40.3)
- moved C7 144.8 mm to (186.3, 36.0)
- moved C8 144.8 mm to (186.3, 38.5)
- moved C9 144.8 mm to (186.3, 41.0)
- moved C6 143.4 mm to (186.2, 43.5)
- moved TP5 142.5 mm to (168.4, 77.7)
- moved C12 138.5 mm to (184.5, 70.5), turned to -90 degrees
- moved JP3 138.2 mm to (189.3, 63.0), turned to 180 degrees
- moved D5 136.7 mm to (162.0, 94.0), turned to 90 degrees
- moved C13 135.6 mm to (181.9, 70.5), turned to -90 degrees
- moved TP3 134.6 mm to (153.0, 95.0)
- moved R9 134.1 mm to (189.2, 66.0), turned to 180 degrees
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Connections:
- C12 pad 1: +BATT -> +12V
- C13 pad 1: +BATT -> +12V
- C14 pad 1: +BATT -> +12V
- C15 pad 1: +BATT -> +12V
- U2 pad 1: GND -> +12V
- U2 pad 3: +BATT -> GND
- U2 pad 4: /5V_FB -> Net-(U2-BOOT)
- U2 pad 6: Net-(U2-BOOT) -> /5V_FB
Routing:
- net /12V_EN: track 0.00 -> 84.2 mm, vias 0 -> 1
- net /5V_EN: track 0.00 -> 56.3 mm, vias 0 -> 2
- net /Vin_EN: track 0.00 -> 48.3 mm, vias 0 -> 2
- net +5V: track 0.00 -> 48.0 mm, vias 0 -> 1
- net /12V_PG_Gate: track 0.00 -> 26.9 mm
- net /Vin: track 1.67 -> 27.4 mm
- net /12V_PG: track 0.00 -> 24.9 mm, vias 0 -> 1
- net Net-(D2-A): track 0.00 -> 23.3 mm, vias 0 -> 1
- net /OV: track 0.00 -> 15.0 mm, vias 0 -> 2
- net /5V_FB: track 0.00 -> 14.7 mm
- net /RAW_BATT: track 0.00 -> 12.2 mm
- net Net-(U2-SW): track 0.00 -> 11.8 mm, vias 0 -> 2
- net Net-(D2-K): track 0.00 -> 10.9 mm, vias 0 -> 1
- net /Gate: track 20.0 -> 27.4 mm
- net +12V: track 0.00 -> 5.78 mm
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- added copper zone on F.Cu, net +12V
- added copper zone on F.Cu, net +5V
- added copper zone on F.Cu, net +BATT
- added copper zone on F.Cu, net /RAW_BATT
- added copper zone on B.Cu, net GND
- added copper zone on F.Cu, net GND
- added copper zone on F.Cu, net Net-(U2-SW)
Other:
- board outline added: 94 x 98 mm

Commit message: PCB Rev 1 Ordered
Parts:
- R1: value 1.9k -> 1.89k
- moved TP2 0.55 mm to (185.0, 24.4)
- moved J5 0.50 mm to (152.5, 89.0)
Changed lines of the file:
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@@
 			(outputformat 1)
 			(mirror no)
-			(drillshape 1)
+			(drillshape 0)
 			(scaleselection 1)
-			(outputdirectory "")
+			(outputdirectory "Manufacture/Rev2/")
 		)
 	)
@@
 	(footprint "PSU-Rev1:KEYSTONE_5002"
 		(layer "F.Cu")
-		(at 185 25)
+		(at 185 24.45)
 		(property "Reference" "TP2"
 			(at 0.032 -2.2064 0)
@@
 	(footprint "PSU-Rev1:6-pin-connector"
 		(layer "F.Cu")
-		(at 153 88.95)
+		(at 152.5 88.95)
 		(property "Reference" "J5"
 			(at 8 -5 0)
@@
 			)
 		)
-		(property "Value" "1.9k"
+		(property "Value" "1.89k"
 			(at 0 -1.65 90)
 			(layer "B.Fab")
@@
 	)
 	(segment
-		(start 185 25)
-		(end 185 27.25)
+		(start 185 24.45)
+		(end 185 26.7)
 		(width 0.2)
 		(layer "F.Cu")
@@
 		(polygon
 			(pts
-				(xy 186 26.75) (xy 189.75 26.75) (xy 189.75 31) (xy 186 31)
+				(xy 186 26.35) (xy 189.75 26.35) (xy 189.75 31) (xy 186 31)
 			)
 		)
@@
 		(polygon
 			(pts
-				(xy 161.5 67.5) (xy 152 67.5) (xy 152 92) (xy 156.5 92) (xy 156.5 74.5) (xy 161.5 74.5)
+				(xy 161.5 67.5) (xy 151 67.5) (xy 151 92) (xy 156.5 92) (xy 156.5 74.5) (xy 161.5 74.5)
 			)
 		)
@@
 		(polygon
 			(pts
-				(xy 169.75 34.5) (xy 169.75 26.75) (xy 186.25 26.75) (xy 186.25 30.75) (xy 174 30.75) (xy 174 34.5)
+				(xy 169.55 34.7) (xy 169.55 26.35) (xy 186.25 26.35) (xy 186.25 30.75) (xy 174 30.75) (xy 174 34.7)
 			)
 		)
